File: EuroESP32.sch (EAGLE design)
At the start: 127 parts, among them IC1 TL074D, IC10 MCP6004, IC2 TL072, IC3 TL072, IC4 WM8731, IC5 TL074D, IC7 ADP7118, P4 POWER_SIMPLE10, U1 LM4040SOT23, U2 MCP3204-CI/SL

Commit message: v0.1
TODO : TLC for the Labels
Parts:
- removed H2: PCB_SCREW, parts_aman:PCB_SCREW
- -10VREF: value -10VREF -> -10V
- CVIN(100K)0: value CVIN(100k)0 -> CVI0
- CVIN(100K)1: value CVIN(100K)1 -> CVI1
- CVIN(100K)2: value CVIN(100K)2 -> CVI2
- CVIN(100K)3: value CVIN(100K)3 -> CVI3
- CVOUT1: value CVOUT1 -> CVO1
- CVOUT2: value CVOUT2 -> CVO2
- CVOUT3: value CVOUT3 -> CVO3
- CVOUT4: value CVOUT4 -> CVO4
Other:
- moved on the sheet: +12V, +3.3VA, -12V, C1, C11, C14, C17, C18, C19, C20, C23, C24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
